Commit message: 16 1 23

File: src/vp_one/description/gazebo_control.xacro (robot description, xacro)
@@ -11,10 +11,10 @@
             <max_wheel_torque>200</max_wheel_torque>
             <max_wheel_acceleration>3.0</max_wheel_acceleration>
-            <!-- Output -->
+            <!-- Output
             <odometry_frame>odom</odometry_frame>
             <robot_base_frame>base_link</robot_base_frame>
-            <publish_odom>true</publish_odom>
+            <publish_odom>false</publish_odom>
             <publish_odom_tf>true</publish_odom_tf>
-            <publish_wheel_tf>true</publish_wheel_tf>
+            <publish_wheel_tf>true</publish_wheel_tf>-->
         </plugin>
     </gazebo>

File: src/vp_one/description/robot.urdf.xacro (robot description, xacro)
@@ -2,5 +2,5 @@
 <robot xmlns:xacro="http://www.ros.org/wiki/xacro"  name="robot">
     <xacro:include filename="robot_core.xacro" />
-    <xacro:include filename="gazebo_control.xacro" />
+    <xacro:include filename="gazebo_control.xacro"/>
     <xacro:include filename="lidar.xacro" />
 </robot>

File: src/vp_one/description/robot_core.xacro (robot description, xacro)
@@ -17,6 +17,22 @@
         <color rgba="1 0 0 1"/>
     </material>
+    <link name="odom">
+    </link>
+    <joint name="base_link_joint" type="fixed">
+        <parent link="odom"/>
+        <child link="base_link"/>
+        <origin xyz="0 0 0" rpy="0 0 0"/>
+    </joint>
     <link name="base_link">
     </link>
+    <!-- ODOM LINK
+    <joint name="odom_joint" type="fixed">
+        <parent link="odom"/>
+        <child link="base_link"/>
+        <origin xyz="0 0 0" rpy="0 0 0"/>
+    </joint>
+    <link name="odom">
+    </link>-->
+   <!--  CHASSIS LINK -->
     <joint name="chassis_joint" type="fixed">
     <parent link="base_link"/>
@@ -47,7 +63,7 @@
     <!-- LEFT WHEEL -->
     <joint name="left_wheel_joint" type="continuous">
-        <parent link="base_link"/>
+        <parent link="chassis"/>
         <child link="left_wheel"/>
-        <origin xyz="0 -0.28 0.06" rpy="${-pi/2} 0 0"/>
+        <origin xyz="0 0.28 0.06" rpy="${-pi/2} 0 0"/>
         <axis xyz="0 0 1"/>
     </joint>
@@ -74,7 +90,7 @@
     <!-- RIGHT WHEEL -->
     <joint name="right_wheel_joint" type="continuous">
-        <parent link="base_link"/>
+        <parent link="chassis"/>
         <child link="right_wheel"/>
-        <origin xyz="0 0.28 0.06" rpy="${pi/2} 0 0"/>
+        <origin xyz="0 -0.28 0.06" rpy="${pi/2} 0 0"/>
         <axis xyz="0 0 -1"/>
     </joint>

Commit message: 19 1 23

File: src/vp_one/description/gazebo_control.xacro (robot description, xacro)
@@ -11,10 +11,10 @@
             <max_wheel_torque>200</max_wheel_torque>
             <max_wheel_acceleration>3.0</max_wheel_acceleration>
-            <!-- Output
+            <!-- Output -->
             <odometry_frame>odom</odometry_frame>
             <robot_base_frame>base_link</robot_base_frame>
-            <publish_odom>false</publish_odom>
+            <publish_odom>true</publish_odom>
             <publish_odom_tf>true</publish_odom_tf>
-            <publish_wheel_tf>true</publish_wheel_tf>-->
+            <publish_wheel_tf>true</publish_wheel_tf>
         </plugin>
     </gazebo>

File: src/vp_one/description/robot_core.xacro (robot description, xacro)
@@ -17,7 +17,7 @@
         <color rgba="1 0 0 1"/>
     </material>
-    <link name="odom">
+    <link name="base_link">
     </link>
-    <joint name="base_link_joint" type="fixed">
+    <!-- <joint name="base_link_joint" type="fixed">
         <parent link="odom"/>
         <child link="base_link"/>
@@ -25,5 +25,5 @@
     </joint>
     <link name="base_link">
-    </link>
+    </link> -->
     <!-- ODOM LINK
     <joint name="odom_joint" type="fixed">
@@ -62,5 +62,5 @@
     </gazebo>
     <!-- LEFT WHEEL -->
-    <joint name="left_wheel_joint" type="continuous">
+    <joint name="joint1" type="continuous">
         <parent link="chassis"/>
         <child link="left_wheel"/>
@@ -88,5 +88,5 @@
     </gazebo>
     <!-- RIGHT WHEEL -->
-    <joint name="right_wheel_joint" type="continuous">
+    <joint name="joint0" type="continuous">
         <parent link="chassis"/>
         <child link="right_wheel"/>
