Commit message: tutto oggi e ieri ok

File: src/vp_one/description/lidar.xacro (robot description, xacro)
@@ -7,49 +7,49 @@
     </joint>
     <link name="laser_frame">
-    <visual>
-        <geometry>
-            <cylinder radius="0.05" length="0.04"/>
-        </geometry>
-        <material name="red"/>
-    </visual>
-    <collision>
-        <geometry>
-            <cylinder radius="0.05" length="0.04"/>
-        </geometry>
-    </collision>
-    <xacro:inertial_cylinder mass="0.1" length="0.04" radius="0.05">
-        <origin xyz="0 0 0" rpy="0 0 0"/>
-    </xacro:inertial_cylinder>
-</link>
-<gazebo reference="laser_frame">
-    <material>Gazebo/Red</material>
-    <sensor name="laser" type="ray">
-    <pose> 0 0 0 0 0 0 </pose>
-    <visualize>true</visualize>
-    <update_rate>10</update_rate>
-    <ray>
-    <scan>
-        <horizontal>
-            <samples>360</samples>
-            <min_angle>-3.14</min_angle>
-            <max_angle>3.14</max_angle>
-        </horizontal>
-    </scan>
-    <range>
-        <min>0.3</min>
-        <max>12</max>
-    </range>
-    </ray>
-    <plugin name="laser_controller" filename="libgazebo_ros_ray_sensor.so">
-    <ros>
-        <argument>~/out:=scan</argument>
-    </ros>
-    <output_type>sensor_msgs/LaserScan</output_type>
-    <frame_name>laser_frame</frame_name>
-</plugin>
-</sensor>
-</gazebo>
-<material name="red">
-    <color rgba="1 0 0 1"/>
-</material>
+        <visual>
+            <geometry>
+                <cylinder radius="0.05" length="0.04"/>
+            </geometry>
+            <material name="red"/>
+        </visual>
+        <collision>
+            <geometry>
+                <cylinder radius="0.05" length="0.04"/>
+            </geometry>
+        </collision>
+        <xacro:inertial_cylinder mass="0.1" length="0.04" radius="0.05">
+            <origin xyz="0 0 0" rpy="0 0 0"/>
+        </xacro:inertial_cylinder>
+    </link>
+    <gazebo reference="laser_frame">
+        <material>Gazebo/Red</material>
+        <sensor name="laser" type="ray">
+            <pose> 0 0 0 0 0 0 </pose>
+            <visualize>true</visualize>
+            <update_rate>10</update_rate>
+            <ray>
+                <scan>
+                    <horizontal>
+                        <samples>360</samples>
+                        <min_angle>-3.14</min_angle>
+                        <max_angle>3.14</max_angle>
+                    </horizontal>
+                </scan>
+                <range>
+                    <min>0.3</min>
+                    <max>12</max>
+                </range>
+            </ray>
+            <plugin name="laser_controller" filename="libgazebo_ros_ray_sensor.so">
+                <ros>
+                    <argument>~/out:=scan</argument>
+                </ros>
+                <output_type>sensor_msgs/LaserScan</output_type>
+                <frame_name>laser_frame</frame_name>
+            </plugin>
+        </sensor>
+    </gazebo>
+    <material name="red">
+        <color rgba="1 0 0 1"/>
+    </material>
 </robot>

File: src/vp_one/description/robot.urdf.xacro (robot description, xacro)
@@ -1,7 +1,7 @@
 <?xml version="1.0"?>
 <robot xmlns:xacro="http://www.ros.org/wiki/xacro"  name="robot">
-    <xacro:include filename="ros2_control.xacro" />
+    <!--<xacro:include filename="ros2_control.xacro" />-->
     <xacro:include filename="robot_core.xacro" />
-    <xacro:include filename="lidar.xacro" />
-    <!-- <xacro:include filename="gazebo_control.xacro" />-->
+    <!--<xacro:include filename="lidar.xacro" />
+    <xacro:include filename="gazebo_control.xacro" />-->
 </robot>

File: src/vp_one/description/ros2_control.xacro (robot description, xacro)
@@ -1,3 +1,3 @@
-<?xml version="1.0"?>
+<!--<?xml version="1.0"?>
 <robot xmlns:xacro="http://www.ros.org/wiki/xacro">
 <ros2_control name="RealRobot" type="system">
@@ -56,3 +56,3 @@
     </plugin>
 </gazebo>
-</robot>
+</robot>-->

Commit message: CODICE SISTEMATO

File: src/vp_one/description/lidar.xacro (robot description, xacro)
@@ -50,6 +50,3 @@
         </sensor>
     </gazebo>
-    <material name="red">
-        <color rgba="1 0 0 1"/>
-    </material>
 </robot>

File: src/vp_one/description/robot.urdf.xacro (robot description, xacro)
@@ -1,7 +1,6 @@
 <?xml version="1.0"?>
 <robot xmlns:xacro="http://www.ros.org/wiki/xacro"  name="robot">
-    <!--<xacro:include filename="ros2_control.xacro" />-->
     <xacro:include filename="robot_core.xacro" />
-    <!--<xacro:include filename="lidar.xacro" />
-    <xacro:include filename="gazebo_control.xacro" />-->
+    <xacro:include filename="gazebo_control.xacro" />
+    <xacro:include filename="lidar.xacro" />
 </robot>

File: src/vp_one/description/robot_core.xacro (robot description, xacro)
@@ -13,4 +13,7 @@
     <material name="black">
         <color rgba="0 0 0 1"/>
+    </material>
+    <material name="red">
+        <color rgba="1 0 0 1"/>
     </material>
     <link name="base_link">
@@ -44,78 +47,78 @@
     <!-- LEFT WHEEL -->
     <joint name="left_wheel_joint" type="continuous">
-    <parent link="base_link"/>
-    <child link="left_wheel"/>
-    <origin xyz="0 0.28 0.06" rpy="-${pi/2} 0 0"/>
-    <axis xyz="0 0 1"/>
+        <parent link="base_link"/>
+        <child link="left_wheel"/>
+        <origin xyz="0 0.28 0.06" rpy="-${pi/2} 0 0"/>
+        <axis xyz="0 0 1"/>
     </joint>
     <link name="left_wheel">
-    <visual>
-        <geometry>
-            <cylinder length="0.06" radius="0.085" />/>
-        </geometry>
-        <material name="black"/>
-    </visual>
-    <collision>
-        <geometry>
-            <cylinder length="0.06" radius="0.085" />/>
-        </geometry>
-        <material name="black"/>
-    </collision>
-    <xacro:inertial_cylinder mass="0.1" length="0.06" radius="0.085">
-        <origin xyz="0 0 0" rpy="0 0 0"/>
-    </xacro:inertial_cylinder>
+        <visual>
+            <geometry>
+                <cylinder length="0.06" radius="0.085" />/>
+            </geometry>
+            <material name="black"/>
+        </visual>
+        <collision>
+            <geometry>
+                <cylinder length="0.06" radius="0.085" />/>
+            </geometry>
+            <material name="black"/>
+        </collision>
+        <xacro:inertial_cylinder mass="0.1" length="0.06" radius="0.085">
+            <origin xyz="0 0 0" rpy="0 0 0"/>
+        </xacro:inertial_cylinder>
     </link>
     <gazebo reference="left_wheel">
-    <material>Gazebo/Black</material>
+        <material>Gazebo/Black</material>
     </gazebo>
     <!-- RIGHT WHEEL -->
     <joint name="right_wheel_joint" type="continuous">
-    <parent link="base_link"/>
-    <child link="right_wheel"/>
-    <origin xyz="0 -0.28 0.06" rpy="${pi/2} 0 0"/>
-    <axis xyz="0 0 -1"/>
+        <parent link="base_link"/>
+        <child link="right_wheel"/>
+        <origin xyz="0 -0.28 0.06" rpy="${pi/2} 0 0"/>
+        <axis xyz="0 0 -1"/>
     </joint>
     <link name="right_wheel">
-    <visual>
-        <geometry>
-            <cylinder length="0.06" radius="0.085" />/>
-        </geometry>
-        <material name="black"/>
-    </visual>
-    <collision>
-        <geometry>
-            <cylinder length="0.06" radius="0.085" />/>
-        </geometry>
-        <material name="black"/>
-    </collision>
-    <xacro:inertial_cylinder mass="0.1" length="0.06" radius="0.085">
-        <origin xyz="0 0 0" rpy="0 0 0"/>
-    </xacro:inertial_cylinder>
+        <visual>
+            <geometry>
+                <cylinder length="0.06" radius="0.085" />/>
+            </geometry>
+            <material name="black"/>
+        </visual>
+        <collision>
+            <geometry>
+                <cylinder length="0.06" radius="0.085" />/>
+            </geometry>
+            <material name="black"/>
+        </collision>
+        <xacro:inertial_cylinder mass="0.1" length="0.06" radius="0.085">
+            <origin xyz="0 0 0" rpy="0 0 0"/>
+        </xacro:inertial_cylinder>
     </link>
     <gazebo reference="right_wheel">
-    <material>Gazebo/Black</material>
+        <material>Gazebo/Black</material>
     </gazebo>
     <!-- CASTER WHEEL -->
     <joint name="caster_wheel_joint" type="fixed">
-    <parent link="chassis"/>
-    <child link="caster_wheel"/>
-    <origin xyz="0.45 0 0" rpy="${pi/2} 0 0"/>
+        <parent link="chassis"/>
+        <child link="caster_wheel"/>
+        <origin xyz="0.45 0 0" rpy="${pi/2} 0 0"/>
     </joint>
     <link name="caster_wheel">
-    <visual>
-        <geometry>
-            <cylinder length="0.04" radius="0.065" />/>
-        </geometry>
-        <material name="blue"/>
-    </visual>
-    <collision>
-        <geometry>
-            <cylinder length="0.04" radius="0.065" />/>
-        </geometry>
-        <material name="blue"/>
-    </collision>
-    <xacro:inertial_cylinder mass="0.1" length="0.04" radius="0.065">
-        <origin xyz="0 0 0" rpy="0 0 0"/>
-    </xacro:inertial_cylinder>
+        <visual>
+            <geometry>
+                <cylinder length="0.04" radius="0.065" />/>
+            </geometry>
+            <material name="blue"/>
+        </visual>
+        <collision>
+            <geometry>
+                <cylinder length="0.04" radius="0.065" />/>
+            </geometry>
+            <material name="blue"/>
+        </collision>
+        <xacro:inertial_cylinder mass="0.1" length="0.04" radius="0.065">
+            <origin xyz="0 0 0" rpy="0 0 0"/>
+        </xacro:inertial_cylinder>
     </link>
     <gazebo reference="caster_wheel">

Commit message: 29 3 23

File: src/vp_one/description/lidar.xacro (robot description, xacro)
@@ -22,5 +22,5 @@
         </xacro:inertial_cylinder>
     </link>
-    <gazebo reference="laser_frame">
+    <!--<gazebo reference="laser_frame">
         <material>Gazebo/Red</material>
         <sensor name="laser" type="ray">
@@ -49,4 +49,4 @@
             </plugin>
         </sensor>
-    </gazebo>
+    </gazebo>-->
 </robot>

File: src/vp_one/description/robot.urdf.xacro (robot description, xacro)
@@ -2,5 +2,5 @@
 <robot xmlns:xacro="http://www.ros.org/wiki/xacro"  name="robot">
     <xacro:include filename="robot_core.xacro" />
-    <xacro:include filename="gazebo_control.xacro"/>
+    <!-- <xacro:include filename="gazebo_control.xacro"/>-->
     <xacro:include filename="lidar.xacro" />
 </robot>

File: src/vp_one/description/robot_core.xacro (robot description, xacro)
@@ -17,6 +17,4 @@
         <color rgba="1 0 0 1"/>
     </material>
-    <link name="base_link">
-    </link>
     <!-- <joint name="base_link_joint" type="fixed">
         <parent link="odom"/>
@@ -26,12 +24,15 @@
     <link name="base_link">
     </link> -->
-    <!-- ODOM LINK
-    <joint name="odom_joint" type="fixed">
-        <parent link="odom"/>
-        <child link="base_link"/>
+<!-- ODOM LINK -->
+    <link name="base_link">
+    </link>
+    <!-- BASE_FOOTPRINT LINK-->
+    <joint name="base_footprint_joint" type="fixed">
+        <parent link="base_link"/>
+        <child link="base_footprint"/>
         <origin xyz="0 0 0" rpy="0 0 0"/>
     </joint>
-    <link name="odom">
-    </link>-->
+    <link name="base_footprint">
+    </link>
    <!--  CHASSIS LINK -->
     <joint name="chassis_joint" type="fixed">
