Commit message: 14 1 23

File: src/vp_one/description/robot_core.xacro (robot description, xacro)
@@ -25,23 +25,23 @@
     </joint>
     <link name="chassis">
-    <visual>
-        <origin xyz="0.28 0 0.41" rpy="0 0 0"/>
-        <geometry>
-            <cylinder length="0.7" radius="0.275"/>
-        </geometry>
-        <material name="white"/>
-    </visual>
-    <collision>
-        <origin xyz="0.28 0 0.41" rpy="0 0 0"/>
-        <geometry>
-            <cylinder length="0.7" radius="0.275"/>
-        </geometry>
-    </collision>
-   <xacro:inertial_cylinder mass="0.1" length="0.7" radius="0.275">
-        <origin xyz="0 0 0" rpy="0 0 0"/>
-    </xacro:inertial_cylinder>
+        <visual>
+            <origin xyz="0.28 0 0.41" rpy="0 0 0"/>
+            <geometry>
+                <cylinder length="0.7" radius="0.275"/>
+            </geometry>
+            <material name="white"/>
+        </visual>
+        <collision>
+            <origin xyz="0.28 0 0.41" rpy="0 0 0"/>
+            <geometry>
+                <cylinder length="0,7" radius="0,275"/>
+            </geometry>
+        </collision>
+        <xacro:inertial_cylinder mass="0.1" length="0.7" radius="0.275">
+            <origin xyz="0 0 0" rpy="0 0 0"/>
+        </xacro:inertial_cylinder>
     </link>
     <gazebo reference="chassis">
-    <material>Gazebo/White</material>
+        <material>Gazebo/White</material>
     </gazebo>
     <!-- LEFT WHEEL -->
@@ -49,5 +49,5 @@
         <parent link="base_link"/>
         <child link="left_wheel"/>
-        <origin xyz="0 0.28 0.06" rpy="-${pi/2} 0 0"/>
+        <origin xyz="0 -0.28 0.06" rpy="${-pi/2} 0 0"/>
         <axis xyz="0 0 1"/>
     </joint>
@@ -55,5 +55,5 @@
         <visual>
             <geometry>
-                <cylinder length="0.06" radius="0.085" />/>
+                <cylinder length="0.06" radius="0.085" />
             </geometry>
             <material name="black"/>
@@ -61,5 +61,5 @@
         <collision>
             <geometry>
-                <cylinder length="0.06" radius="0.085" />/>
+                <cylinder length="0.06" radius="0.085" />
             </geometry>
             <material name="black"/>
@@ -76,5 +76,5 @@
         <parent link="base_link"/>
         <child link="right_wheel"/>
-        <origin xyz="0 -0.28 0.06" rpy="${pi/2} 0 0"/>
+        <origin xyz="0 0.28 0.06" rpy="${pi/2} 0 0"/>
         <axis xyz="0 0 -1"/>
     </joint>
@@ -82,5 +82,5 @@
         <visual>
             <geometry>
-                <cylinder length="0.06" radius="0.085" />/>
+                <cylinder length="0.06" radius="0.085" />
             </geometry>
             <material name="black"/>
@@ -88,5 +88,5 @@
         <collision>
             <geometry>
-                <cylinder length="0.06" radius="0.085" />/>
+                <cylinder length="0.06" radius="0.085" />
             </geometry>
             <material name="black"/>
@@ -108,5 +108,5 @@
         <visual>
             <geometry>
-                <cylinder length="0.04" radius="0.065" />/>
+                <cylinder length="0.04" radius="0.065" />
             </geometry>
             <material name="blue"/>
@@ -114,5 +114,5 @@
         <collision>
             <geometry>
-                <cylinder length="0.04" radius="0.065" />/>
+                <cylinder length="0.04" radius="0.065" />
             </geometry>
             <material name="blue"/>

Commit message: ordine

File: src/vp_one/description/robot_core.xacro (robot description, xacro)
@@ -79,5 +79,4 @@
                 <cylinder length="0.06" radius="0.085" />
             </geometry>
-            <material name="black"/>
         </collision>
         <xacro:inertial_cylinder mass="0.1" length="0.06" radius="0.085">
@@ -106,5 +105,4 @@
                 <cylinder length="0.06" radius="0.085" />
             </geometry>
-            <material name="black"/>
         </collision>
         <xacro:inertial_cylinder mass="0.1" length="0.06" radius="0.085">

Commit message: fine 06 04 23

File: src/vp_one/description/robot_core.xacro (robot description, xacro)
@@ -63,5 +63,5 @@
     </gazebo>
     <!-- LEFT WHEEL -->
-    <joint name="joint1" type="continuous">
+    <joint name="joint0" type="continuous">
         <parent link="chassis"/>
         <child link="left_wheel"/>
@@ -89,5 +89,5 @@
     </gazebo>
     <!-- RIGHT WHEEL -->
-    <joint name="joint0" type="continuous">
+    <joint name="joint1" type="continuous">
         <parent link="chassis"/>
         <child link="right_wheel"/>
